File: hardware/joint_boards/STM32F103_microcontroller_board/STM32F103_microcontroller_board.sch (KiCad schematic (older format))
At the start: 29 parts

Commit message: version 1 of MCU schematic
Parts:
- removed J?: Conn_01x03, symbol Connector_Generic:Conn_01x03
- added J?: Conn_02x10_Odd_Even, symbol Connector_Generic:Conn_02x10_Odd_Even
- added J?: Conn_02x09_Counter_Clockwise, symbol Connector_Generic:Conn_02x09_Counter_Clockwise
- added J?: Conn_01x04, symbol Connector_Generic:Conn_01x04
Connections:
- net labels added: Enable, FWD_REV, OSC_IN, OSC_OUT, PA15, PA3, PB0, PB1, PB12, PB2, PB3, PB4, PB5, PB7, PC15, Speed_PWM, U_driver, U_encoder, V_driver, V_encoder, W_driver, W_encoder, as5040_CLK, as5040_CS, as5040_DO, as5040_LSB_PWM, as5040_PROG, as5040_lsb_pwm, local_encoder_pwm
- net labels removed: TIM3CH1
- wire segments 95 -> 105
Other:
- note added: "Connector to Motor Controller board"
- note added: "Questions:\nPin assignment for Input/Output connectors"
- note added: "Status LED\n(blue)"
- note added: "Status LED\n(green)"
- note added: "Unused Pins breakout"
- note removed: "Questions:\nPin assignment for Input/Output connectors\nGround Sheilding for PWM input from AS 5040\nSMT component size for TVS device"
- note removed: "Status LED (blue)"
- note removed: "Status LED (green)"

Commit message: footprints associated and schematic finalized. Most components have sources
Parts:
- C1, C2: renamed from C?; footprint (none) -> Capacitor_SMD:CP_Elec_6.3x5.4; symbol Device:C -> Device:CP1
- C10, C11: renamed from C?; value C -> 100nF; footprint (none) -> Capacitor_SMD:C_0603_1608Metric_Pad1.05x0.95mm_HandSolder
- C3, C4, C5, C6, C7, C8, C9: renamed from C?; footprint (none) -> Capacitor_SMD:C_0603_1608Metric_Pad1.05x0.95mm_HandSolder
- D1: renamed from D?; value LED -> RED LED; footprint (none) -> LED_SMD:LED_0603_1608Metric_Pad1.05x0.95mm_HandSolder
- D2: renamed from D?; value 11DQ06 -> SR106; footprint (none) -> Diode_SMD:D_SOD-323_HandSoldering
- D3: renamed from D?; value LED -> GRN LED; footprint (none) -> LED_SMD:LED_0603_1608Metric_Pad1.05x0.95mm_HandSolder
- D4: renamed from D?; value LED -> BLUE LED; footprint (none) -> LED_SMD:LED_0603_1608Metric_Pad1.05x0.95mm_HandSolder
- D5: renamed from D?; value D_TVS_x2_AAC -> ESDCAN24-2BLY; footprint (none) -> Package_TO_SOT_SMD:SOT-23_Handsoldering
- J1: renamed from J?; footprint (none) -> Connector_PinHeader_2.54mm:PinHeader_2x10_P2.54mm_Vertical
- J2: renamed from J?; footprint (none) -> Connector_PinHeader_2.54mm:PinHeader_1x04_P2.54mm_Horizontal
- J3, J4: renamed from J?; footprint (none) -> Connector_Molex:Molex_KK-254_AE-6410-08A_1x08_P2.54mm_Vertical; symbol Connector_Generic:Conn_01x04 -> Connector_Generic:Conn_01x08
- J5: renamed from J?; footprint (none) -> Connector_PinHeader_2.54mm:PinHeader_1x03_P2.54mm_Vertical
- J6: renamed from J?; footprint (none) -> Connector_PinHeader_2.54mm:PinHeader_2x09_P2.54mm_Vertical
- JP1: renamed from JP?; footprint (none) -> Jumper:SolderJumper-2_P1.3mm_Open_TrianglePad1.0x1.5mm
- L1: renamed from L?; footprint (none) -> Inductor_THT:L_Radial_D8.7mm_P5.00mm_Fastron_07HCP
- R1: renamed from R?; value R -> 33; footprint (none) -> Resistor_SMD:R_0603_1608Metric_Pad1.05x0.95mm_HandSolder
- R2, R3: renamed from R?; value R -> 68; footprint (none) -> Resistor_SMD:R_0603_1608Metric_Pad1.05x0.95mm_HandSolder
- R4: renamed from R?; footprint (none) -> Resistor_SMD:R_0603_1608Metric_Pad1.05x0.95mm_HandSolder
- gave numbers to parts that had none: 3
Connections:
- net labels removed: as5040_lsb_pwm
- wire segments 105 -> 126
- no-connect marks 0 -> 1

Commit message: board layed out after 6 hours
Parts:
- J2: footprint Connector_PinHeader_2.54mm:PinHeader_1x04_P2.54mm_Horizontal -> Connector_PinHeader_2.54mm:PinHeader_1x04_P2.54mm_Vertical
- R1: value 33 -> 68
- R3: value 68 -> 33
Connections:
- net labels added: CAN+, CAN-
- net labels removed: CANH, CANL
- wire segments 126 -> 133
- no-connect marks 1 -> 4
Changed lines of the file:
@@
 Text Label 6100 5150 0    50   ~ 0
 SWCLK
-Wire Wire Line
-	6000 5050 6500 5050
-Wire Wire Line
-	6000 5150 6500 5150
 $Comp
 L power:GND #PWR020
@@
 	1    0    0    -1
 $EndComp
-Wire Wire Line
-	8400 4400 8400 4300
-Wire Wire Line
-	8400 4300 8800 4300
 $Comp
 L Device:C C9
@@
 $EndComp
 Wire Wire Line
-	8400 4900 8800 4900
-Wire Wire Line
-	8400 4500 8400 4900
-Wire Wire Line
 	6000 4950 7150 4950
 Wire Wire Line
@@
 CANRX
 Text Label 9600 4250 0    50   ~ 0
-CANH
+CAN-
 Text Label 9600 4950 0    50   ~ 0
-CANL
+CAN+
 $Comp
 L Device:D_TVS_x2_AAC D5
@@
 Wire Wire Line
 	9100 4250 9450 4250
-Connection ~ 8800 4300
 Wire Wire Line
 	8800 4900 9100 4900
@@
 Wire Wire Line
 	9100 4950 9450 4950
-Connection ~ 8800 4900
 $Comp
 L power:GND #PWR018
@@
 P 4250 1150
 F 0 "R1" V 4043 1150 50  0000 C CNN
-F 1 "33" V 4134 1150 50  0000 C CNN
+F 1 "68" V 4134 1150 50  0000 C CNN
 F 2 "Resistor_SMD:R_0603_1608Metric_Pad1.05x0.95mm_HandSolder" V 4180 1150 50  0001 C CNN
 F 3 "~" H 4250 1150 50  0001 C CNN
@@
 VIN
 Text Label 1050 4750 2    50   ~ 0
-CANH
+CAN+
 Text Label 950  4550 2    50   ~ 0
 EXT_GND
 Text Label 1050 4850 2    50   ~ 0
-CANL
+CAN-
 $Comp
 L Connector_Generic:Conn_01x08 J4
@@
 VIN
 Text Label 2300 4750 2    50   ~ 0
-CANH
+CAN+
 Text Label 2200 4550 2    50   ~ 0
 EXT_GND
 Text Label 2300 4850 2    50   ~ 0
-CANL
+CAN-
 Text Notes 1100 4050 0    50   ~ 0
 Input
@@
 P 3600 3650
 F 0 "R3" H 3400 3650 50  0000 C CNN
-F 1 "68" V 3500 3650 50  0000 C CNN
+F 1 "33" V 3500 3650 50  0000 C CNN
 F 2 "Resistor_SMD:R_0603_1608Metric_Pad1.05x0.95mm_HandSolder" V 3530 3650 50  0001 C CNN
 F 3 "~" H 3600 3650 50  0001 C CNN
@@
 Text Label 6000 4750 0    50   ~ 0
 W_driver
-Text Label 4700 5050 2    50   ~ 0
-as5040_CLK
-Text Label 4700 5150 2    50   ~ 0
-as5040_DO
-Text Label 4700 5250 2    50   ~ 0
-as5040_PROG
 Text Label 4700 4350 2    50   ~ 0
 local_encoder_pwm
@@
 Wire Wire Line
 	2450 5950 2600 5950
-Text Label 1950 6050 2    50   ~ 0
+Text Label 1950 6250 2    50   ~ 0
 OSC_IN
 Text Label 1950 6150 2    50   ~ 0
 OSC_OUT
-Text Label 1950 6250 2    50   ~ 0
+Text Label 1950 6050 2    50   ~ 0
 PC15
-Text Label 1950 6350 2    50   ~ 0
+Text Label 1950 6650 2    50   ~ 0
 PB0
+Text Label 1950 6550 2    50   ~ 0
+PB1
+Text Label 2450 6550 0    50   ~ 0
+PB2
+Text Label 2450 6650 0    50   ~ 0
+PB3
+Text Label 2450 6150 0    50   ~ 0
+PB4
+Text Label 2450 6350 0    50   ~ 0
+PB5
 Text Label 1950 6450 2    50   ~ 0
-PB1
-Text Label 1950 6550 2    50   ~ 0
-PB2
-Text Label 1950 6650 2    50   ~ 0
-PB3
-Text Label 2450 6650 0    50   ~ 0
-PB4
-Text Label 2450 6550 0    50   ~ 0
-PB5
+PB7
 Text Label 2450 6450 0    50   ~ 0
-PB7
-Text Label 2450 6350 0    50   ~ 0
 PB12
 Text Label 6000 4050 0    50   ~ 0
 PA3
-Text Label 2450 6250 0    50   ~ 0
+Text Label 1950 6350 2    50   ~ 0
 PA3
 Text Label 6000 5250 0    50   ~ 0
 PA15
-Text Label 2450 6150 0    50   ~ 0
+Text Label 2450 6250 0    50   ~ 0
 PA15
 $Comp
@@
 F 0 "J2" H 7230 2842 50  0000 L CNN
 F 1 "Conn_01x04" H 7230 2751 50  0000 L CNN
-F 2 "Connector_PinHeader_2.54mm:PinHeader_1x04_P2.54mm_Horizontal" H 7150 2850 50  0001 C CNN
+F 2 "Connector_PinHeader_2.54mm:PinHeader_1x04_P2.54mm_Vertical" H 7150 2850 50  0001 C CNN
 F 3 "~" H 7150 2850 50  0001 C CNN
 	1    7150 2850
@@
 Wire Wire Line
 	1050 4850 1150 4850
+Wire Wire Line
+	8800 4300 8600 4300
+Wire Wire Line
+	8600 4300 8600 4500
+Wire Wire Line
+	8600 4500 8400 4500
+Connection ~ 8800 4300
+Wire Wire Line
+	8800 4900 8500 4900
+Wire Wire Line
+	8500 4900 8500 4400
+Wire Wire Line
+	8500 4400 8400 4400
+Connection ~ 8800 4900
+Wire Wire Line
+	6000 5050 6400 5050
+Wire Wire Line
+	6400 5050 6400 5150
+Wire Wire Line
+	6400 5150 6500 5150
+Wire Wire Line
+	6000 5150 6350 5150
+Wire Wire Line
+	6350 5150 6350 5100
+Wire Wire Line
+	6350 5100 6500 5100
+Wire Wire Line
+	6500 5100 6500 5050
+NoConn ~ 4700 5050
+NoConn ~ 4700 5150
+NoConn ~ 4700 5250
 $EndSCHEMATC
