File: hardware/joint_boards/STM32F103_microcontroller_board/STM32F103_microcontroller_board.kicad_pcb (KiCad board)
At the start: 2 copper layers, 44.4 x 44.4 mm, 35 parts, among them J1 Conn_02x10_Odd_Even, J2 Conn_01x04, J3 Conn_01x04, J4 Conn_01x04, J5 Conn_01x03, J6 Conn_02x09_Counter_Clockwise, U1 LM2574HVM-3.3, U2 STM32F103CBTx, U3 SN65HVD232

Commit message: basic schematic setup for driver board
Other:
- board text added: "Open Source Robot Joint STM32F103CBT6 Controll Board Version 1.2018.11.13 Designer: Cole Mortensen Docs on gitlab.com/magicole/OSRJ"
Changed lines of the file:
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@@
   (general
     (thickness 1.6)
-    (drawings 13)
+    (drawings 14)
     (tracks 698)
     (zones 0)
@@
   (page USLetter)
   (layers
-    (0 F.Cu signal)
-    (31 B.Cu signal)
+    (0 F.Cu signal hide)
+    (31 B.Cu signal hide)
     (32 B.Adhes user hide)
     (33 F.Adhes user hide)
     (34 B.Paste user)
-    (35 F.Paste user)
+    (35 F.Paste user hide)
     (36 B.SilkS user)
-    (37 F.SilkS user)
+    (37 F.SilkS user hide)
     (38 B.Mask user)
-    (39 F.Mask user)
+    (39 F.Mask user hide)
     (40 Dwgs.User user)
     (41 Cmts.User user hide)
@@
     (45 Margin user)
     (46 B.CrtYd user)
-    (47 F.CrtYd user)
+    (47 F.CrtYd user hide)
     (48 B.Fab user hide)
     (49 F.Fab user hide)
@@
     (tags "Capacitor Electrolytic")
     (attr smd)
-    (fp_text reference C1 (at 4.6 -2.6 180) (layer F.SilkS)
+    (fp_text reference C1 (at 0.15 4.2 180) (layer F.SilkS)
       (effects (font (size 1 1) (thickness 0.15)))
     )
@@
     (tags "Capacitor Electrolytic")
     (attr smd)
-    (fp_text reference C2 (at 0.2 2.1 180) (layer F.SilkS)
+    (fp_text reference C2 (at 4.15 1.95 180) (layer F.SilkS)
       (effects (font (size 1 1) (thickness 0.15)))
     )
@@
     (tags "capacitor handsolder")
     (attr smd)
-    (fp_text reference C3 (at 2.9 0.25) (layer F.SilkS)
+    (fp_text reference C3 (at 2.65 -0.1) (layer F.SilkS)
       (effects (font (size 1 1) (thickness 0.15)))
     )
@@
     (tags "capacitor handsolder")
     (attr smd)
-    (fp_text reference C4 (at 2.35 -0.3) (layer F.SilkS)
+    (fp_text reference C4 (at 2.25 -0.1) (layer F.SilkS)
       (effects (font (size 1 1) (thickness 0.15)))
     )
@@
     (tags "capacitor handsolder")
     (attr smd)
-    (fp_text reference C7 (at -2.45 -0.05 180) (layer F.SilkS)
+    (fp_text reference C7 (at -3.35 0.2 270) (layer F.SilkS)
       (effects (font (size 1 1) (thickness 0.15)))
     )
@@
     (tags "capacitor handsolder")
     (attr smd)
-    (fp_text reference C8 (at -2.5 -0.4 180) (layer F.SilkS)
+    (fp_text reference C8 (at -2.5 -0.4 270) (layer F.SilkS)
       (effects (font (size 1 1) (thickness 0.15)))
     )
@@
     (tags "capacitor handsolder")
     (attr smd)
-    (fp_text reference C9 (at 0 -1.43 180) (layer F.SilkS)
+    (fp_text reference C9 (at 0 -1.65 180) (layer F.SilkS)
       (effects (font (size 1 1) (thickness 0.15)))
     )
@@
     (descr "Molex KK-254 Interconnect System, old/engineering part number: AE-6410-08A example for new part number: 22-27-2081, 8 Pins (http://www.molex.com/pdm_docs/sd/022272021_sd.pdf), generated with kicad-footprint-generator")
     (tags "connector Molex KK-254 side entry")
-    (fp_text reference J3 (at -2.4 -2.8) (layer F.SilkS)
+    (fp_text reference J3 (at -2.37 -0.6) (layer F.SilkS)
       (effects (font (size 1 1) (thickness 0.15)))
     )
@@
     (descr "Molex KK-254 Interconnect System, old/engineering part number: AE-6410-08A example for new part number: 22-27-2081, 8 Pins (http://www.molex.com/pdm_docs/sd/022272021_sd.pdf), generated with kicad-footprint-generator")
     (tags "connector Molex KK-254 side entry")
-    (fp_text reference J4 (at 20.4 0 90) (layer F.SilkS)
+    (fp_text reference J4 (at 20.4 0 180) (layer F.SilkS)
       (effects (font (size 1 1) (thickness 0.15)))
     )
@@
     (descr "Through hole straight pin header, 2x09, 2.54mm pitch, double rows")
     (tags "Through hole pin header THT 2x09 2.54mm double row")
-    (fp_text reference J6 (at 1.27 -2.33 90) (layer F.SilkS)
+    (fp_text reference J6 (at 3.05 -2.33 180) (layer F.SilkS)
       (effects (font (size 1 1) (thickness 0.15)))
     )
@@
     (descr "Inductor, Radial series, Radial, pin pitch=5.00mm, , diameter=8.7mm, Fastron, 07HCP, http://cdn-reichelt.de/documents/datenblatt/B400/DS_07HCP.pdf")
     (tags "Inductor Radial series Radial pin pitch 5.00mm  diameter 8.7mm Fastron 07HCP")
-    (fp_text reference L1 (at 2.4 -0.1) (layer F.SilkS)
+    (fp_text reference L1 (at -1.95 -3.05) (layer F.SilkS)
       (effects (font (size 1 1) (thickness 0.15)))
     )
@@
     (tags "SOIC 1.27")
     (attr smd)
-    (fp_text reference U1 (at 0 -0.2) (layer F.SilkS)
+    (fp_text reference U1 (at 4.95 -5.05) (layer F.SilkS)
       (effects (font (size 1 1) (thickness 0.15)))
     )
@@
     (tags "QFP 0.5")
     (attr smd)
-    (fp_text reference U2 (at -0.15 0.2) (layer F.SilkS)
+    (fp_text reference U2 (at 4.1 -4.4) (layer F.SilkS)
       (effects (font (size 1 1) (thickness 0.15)))
     )
@@
     (tags "mounting hole 3.2mm no annular m3")
     (attr virtual)
-    (fp_text reference REF** (at 0 -4.2) (layer F.SilkS)
+    (fp_text reference REF** (at 0 -4.2) (layer F.SilkS) hide
       (effects (font (size 1 1) (thickness 0.15)))
     )
@@
     (tags "mounting hole 3.2mm no annular m3")
     (attr virtual)
-    (fp_text reference REF** (at 0 -4.2) (layer F.SilkS)
+    (fp_text reference REF** (at 0 -4.2) (layer F.SilkS) hide
       (effects (font (size 1 1) (thickness 0.15)))
     )
@@
     (tags "mounting hole 3.2mm no annular m3")
     (attr virtual)
-    (fp_text reference REF** (at 0 -4.2) (layer F.SilkS)
+    (fp_text reference REF** (at -1.55 -3.9) (layer F.SilkS) hide
       (effects (font (size 1 1) (thickness 0.15)))
     )
@@
     (tags "mounting hole 3.2mm no annular m3")
     (attr virtual)
-    (fp_text reference REF** (at 0 -4.2) (layer F.SilkS)
+    (fp_text reference REF** (at 0 -4.2) (layer F.SilkS) hide
       (effects (font (size 1 1) (thickness 0.15)))
     )
@@
     (pad 1 np_thru_hole circle (at 0 0) (size 3.2 3.2) (drill 3.2) (layers *.Cu *.Mask))
   )
+  (gr_text "Open Source Robot Joint \nSTM32F103CBT6\nControll Board\nVersion 1.2018.11.13\nDesigner:\nCole Mortensen\nDocs on gitlab.com/magicole/OSRJ" (at 145.35 76.9) (layer B.SilkS)
+    (effects (font (size 1.2 1.2) (thickness 0.2)) (justify left mirror))
+  )
   (gr_line (start 107.55 98.6) (end 107.55 61.35) (layer Edge.Cuts) (width 0.15))
